Commit message: Adjusted axis of rotation for wheels

File: prius_description/urdf/prius.urdf (robot description, URDF)
Before this commit: robot prius, 7 links, 6 joints
Joints:
- joint bl_wheel_joint: axis 0 1 0 -> 1 0 0
- joint br_wheel_joint: axis 0 1 0 -> 1 0 0
- joint fl_steer_joint: limit lower=3.14 upper=3.14 effort=100000000 velocity=1000000 -> (none); type revolute -> continuous
- joint fl_wheel_joint: axis 0 1 0 -> 1 0 0
- joint fr_steer_joint: limit lower=3.14 upper=3.14 effort=100000000 velocity=1000000 -> (none); type revolute -> continuous
- joint fr_wheel_joint: axis 0 1 0 -> 1 0 0

Commit message: Renders on both GZ and RVIZ

File: prius_description/urdf/prius.urdf (robot description, URDF)
Before this commit: robot prius, 7 links, 6 joints
Links:
- link bl_wheel: mass None -> 0.01; geometry collision sphere radius=0.31265
- link br_wheel: mass None -> 0.01; geometry collision sphere radius=0.31265
- link chassis: mass None -> 0.01; geometry collision box size=1.168381 1.654253 0.272347; collision box size=1.267845 1.116344 0.244286
- link fl_axle: mass None -> 0.01
- link fl_wheel: mass None -> 0.01; geometry collision sphere radius=0.31265
- link fr_axle: mass None -> 0.01
- link fr_wheel: mass None -> 0.01; geometry collision sphere radius=0.31265

Commit message: Rename link names, updated inertials, added 5.1 deg of caster to steering joints

File: prius_description/urdf/prius.urdf (robot description, URDF)
Before this commit: robot prius, 7 links, 6 joints
Links:
- removed link bl_wheel
- removed link br_wheel
- removed link fl_wheel
- removed link fr_wheel
- added link front_left_wheel, mass 11; collision sphere radius=0.31265
- added link front_right_wheel, mass 11; collision sphere radius=0.31265
- added link rear_left_wheel, mass 11; collision sphere radius=0.31265
- added link rear_right_wheel, mass 11; collision sphere radius=0.31265
- link chassis: mass 0.01 -> 1356.0
- link fl_axle: mass 0.01 -> 1
- link fr_axle: mass 0.01 -> 1
Joints:
- removed joint bl_wheel_joint
- removed joint br_wheel_joint
- removed joint fl_wheel_joint
- removed joint fr_wheel_joint
- added joint front_left_wheel_joint: type continuous, parent fl_axle, child front_left_wheel, origin xyz=0 0 0 rpy=0 0 0, axis 1 0 0
- added joint front_right_wheel_joint: type continuous, parent fr_axle, child front_right_wheel, origin xyz=0 0 0 rpy=0 0 0, axis 1 0 0
- added joint rear_left_wheel_joint: type continuous, parent chassis, child rear_left_wheel, origin xyz=0.793 1.45 0.3 rpy=0 0 0, axis 1 0 0
- added joint rear_right_wheel_joint: type continuous, parent chassis, child rear_right_wheel, origin xyz=-0.793 1.45 0.3 rpy=0 0 0, axis 1 0 0
- joint fl_steer_joint: origin xyz=0.767 -1.41 0.3 rpy=0 0 0 -> xyz=0.767 -1.41 0.3 rpy=-0.089 0 0
- joint fr_steer_joint: origin xyz=-0.767 -1.41 0.3 rpy=0 0 0 -> xyz=-0.767 -1.41 0.3 rpy=-0.089 0 0

Commit message: Surface properties for wheels

File: prius_description/urdf/prius.urdf (robot description, URDF)
Before this commit: robot prius, 7 links, 6 joints
Links:
- added link steering_wheel, mass 1.0; visual cylinder length=0.01 radius=0.16
Joints:
- added joint steering_joint: type continuous, parent chassis, child steering_wheel, origin xyz=0.44 -0.717609 0.938807 rpy=-0.87 0 0, axis 0 1 0.84365

Commit message: Can teleop car

File: prius_description/urdf/prius.urdf (robot description, URDF)
Before this commit: robot prius, 8 links, 7 joints
Joints:
- removed joint fl_steer_joint
- removed joint fr_steer_joint
- added joint front_left_steer_joint: type continuous, parent chassis, child fl_axle, origin xyz=0.767 -1.41 0.3 rpy=-0.089 0 0, axis 0 0 1
- added joint front_right_steer_joint: type continuous, parent chassis, child fr_axle, origin xyz=-0.767 -1.41 0.3 rpy=-0.089 0 0, axis 0 0 1

Commit message: Steering works

File: prius_description/urdf/prius.urdf (robot description, URDF)
Before this commit: robot prius, 8 links, 7 joints
Joints:
- joint front_left_steer_joint: limit (none) -> lower=-0.8727 upper=0.8727 effort=10000000 velocity=1000000
- joint front_right_steer_joint: limit (none) -> lower=-0.8727 upper=0.8727 effort=10000000 velocity=1000000
- joint steering_joint: axis 0 1 0.84365 -> 0 0 1; limit (none) -> lower=-7.85 upper=7.85 effort=10000000 velocity=1000000

Commit message: laserscan displayed in rviz

File: prius_description/urdf/prius.urdf (robot description, URDF)
Before this commit: robot prius, 8 links, 7 joints
Links:
- added link front_laser_link
Joints:
- added joint front_laser_joint: type fixed, parent chassis, child front_laser_link, origin xyz=0 -2.4 0.5 rpy=0 0.05 -1.5707

Commit message: Two more front laser sensors

File: prius_description/urdf/prius.urdf (robot description, URDF)
Before this commit: robot prius, 9 links, 8 joints
Links:
- added link front_left_laser_link, mass 1
- added link front_right_laser_link, mass 1
- link front_laser_link: mass None -> 1
Joints:
- added joint front_left_laser_joint: type fixed, parent chassis, child front_left_laser_link, origin xyz=1 -2.3 0.5 rpy=0 0.05 0
- added joint front_right_laser_joint: type fixed, parent chassis, child front_right_laser_link, origin xyz=-1 -2.3 0.5 rpy=0 0.05 3.14

Commit message: add base_link re: REP 105 http://www.ros.org/reps/rep-0105.html

File: prius_description/urdf/prius.urdf (robot description, URDF)
Before this commit: robot prius, 11 links, 10 joints
Links:
- added link base_link, mass 1
Joints:
- added joint base_link_connection: type fixed, parent base_link, child chassis, origin xyz=1.45 0 0 rpy=0 0 1.57, axis 1 0 0

Commit message: Added lasers and cameras to the car

File: prius_description/urdf/prius.urdf (robot description, URDF)
Before this commit: robot prius, 12 links, 11 joints
Links:
- removed link front_laser_link
- added link back_camera_link, mass 1
- added link center_laser_link, mass 1
- added link front_camera_link, mass 1
- added link left_camera_link, mass 1
- added link right_camera_link, mass 1
Joints:
- removed joint front_laser_joint
- added joint back_camera_joint: type fixed, parent chassis, child back_camera_link, origin xyz=0 1.45 1.4 rpy=0 0.05 1.5707
- added joint center_laser_joint: type fixed, parent chassis, child center_laser_link, origin xyz=0 0.4 1.8 rpy=0 0 -1.5707
- added joint front_camera_joint: type fixed, parent chassis, child front_camera_link, origin xyz=0 -0.4 1.4 rpy=0 0.05 -1.5707
- added joint left_camera_joint: type fixed, parent chassis, child left_camera_link, origin xyz=1 -0.7 1.0 rpy=0 0.05 1.0
- added joint right_camera_joint: type fixed, parent chassis, child right_camera_link, origin xyz=-1 -0.7 1.0 rpy=0 0.05 2.1416

Commit message: Added 8 range sensors

File: prius_description/urdf/prius.urdf (robot description, URDF)
Before this commit: robot prius, 16 links, 15 joints
Links:
- added link back_left_far_sonar_link, mass 1
- added link back_left_middle_sonar_link, mass 1
- added link back_right_far_sonar_link, mass 1
- added link back_right_middle_sonar_link, mass 1
- added link front_left_far_sonar_link, mass 1
- added link front_left_middle_sonar_link, mass 1
- added link front_right_far_sonar_link, mass 1
- added link front_right_middle_sonar_link, mass 1
Joints:
- added joint back_left_far_sonar_joint: type fixed, parent chassis, child back_left_far_sonar_link, origin xyz=0.7 2.4 0.5 rpy=0 0 1.5707
- added joint back_left_middle_sonar_joint: type fixed, parent chassis, child back_left_middle_sonar_link, origin xyz=0.24 2.4 0.5 rpy=0 0 1.5707
- added joint back_right_far_sonar_joint: type fixed, parent chassis, child back_right_far_sonar_link, origin xyz=-0.7 2.4 0.5 rpy=0 0 1.5707
- added joint back_right_middle_sonar_joint: type fixed, parent chassis, child back_right_middle_sonar_link, origin xyz=-0.24 2.4 0.5 rpy=0 0 1.5707
- added joint front_left_far_sonar_joint: type fixed, parent chassis, child front_left_far_sonar_link, origin xyz=0.7 -2.1 0.5 rpy=0 0 -1.5707
- added joint front_left_middle_sonar_joint: type fixed, parent chassis, child front_left_middle_sonar_link, origin xyz=0.24 -2.3 0.5 rpy=0 0 -1.5707
- added joint front_right_far_sonar_joint: type fixed, parent chassis, child front_right_far_sonar_link, origin xyz=-0.7 -2.1 0.5 rpy=0 0 -1.5707
- added joint front_right_middle_sonar_joint: type fixed, parent chassis, child front_right_middle_sonar_link, origin xyz=-0.24 -2.3 0.5 rpy=0 0 -1.5707

Commit message: Added sky, removed caster angle

File: prius_description/urdf/prius.urdf (robot description, URDF)
Before this commit: robot prius, 24 links, 23 joints
Joints:
- joint front_left_steer_joint: origin xyz=0.767 -1.41 0.3 rpy=-0.089 0 0 -> xyz=0.767 -1.41 0.3 rpy=0 0 0
- joint front_right_steer_joint: origin xyz=-0.767 -1.41 0.3 rpy=-0.089 0 0 -> xyz=-0.767 -1.41 0.3 rpy=0 0 0

Commit message: Wheel visuals now move in gazebo and rviz

File: prius_description/urdf/prius.urdf (robot description, URDF)
Before this commit: robot prius, 24 links, 23 joints
Links:
- link chassis: geometry collision box size=1.168381 1.654253 0.272347; collision box size=1.267845 1.116344 0.244286
- link front_left_wheel: geometry collision sphere radius=0.31265; visual mesh filename=package://prius_description/meshes/wheel.obj scale=0.01 0.01 0.01
- link front_right_wheel: geometry collision sphere radius=0.31265; visual mesh filename=package://prius_description/meshes/wheel.obj scale=0.01 0.01 0.01
- link rear_left_wheel: geometry collision sphere radius=0.31265; visual mesh filename=package://prius_description/meshes/wheel.obj scale=0.01 0.01 0.01
- link rear_right_wheel: geometry collision sphere radius=0.31265; visual mesh filename=package://prius_description/meshes/wheel.obj scale=0.01 0.01 0.01
- link steering_wheel: geometry visual mesh filename=package://prius_description/meshes/steering_wheel.obj scale=0.01 0.01 0.01

Commit message: Fix the steering wheel position

File: prius_description/urdf/prius.urdf (robot description, URDF)
Before this commit: robot prius, 24 links, 23 joints
Joints:
- joint steering_joint: origin xyz=0.44 -0.717609 0.938807 rpy=-0.87 0 0 -> xyz=0.357734 -0.627868 0.988243 rpy=-1.302101 0 0

Commit message: Update base_link to be under rear axle
This is more standard.
Fixes #16

File: prius_description/urdf/prius.urdf (robot description, URDF)
Before this commit: robot prius, 24 links, 23 joints
Joints:
- joint base_link_connection: origin xyz=1.45 0 0 rpy=0 0 0 -> xyz=1.45 0 0 rpy=0 0 1.57

Commit message: Removing sonars, 3d Lidar and limiting to one 2d lidar

File: prius_description/urdf/prius.urdf (robot description, URDF)
Before this commit: robot prius, 24 links, 23 joints
Links:
- removed link back_left_far_sonar_link
- removed link back_left_middle_sonar_link
- removed link back_right_far_sonar_link
- removed link back_right_middle_sonar_link
- removed link center_laser_link
- removed link front_left_far_sonar_link
- removed link front_left_middle_sonar_link
- removed link front_right_far_sonar_link
- removed link front_right_laser_link
- removed link front_right_middle_sonar_link
Joints:
- removed joint back_left_far_sonar_joint
- removed joint back_left_middle_sonar_joint
- removed joint back_right_far_sonar_joint
- removed joint back_right_middle_sonar_joint
- removed joint center_laser_joint
- removed joint front_left_far_sonar_joint
- removed joint front_left_middle_sonar_joint
- removed joint front_right_far_sonar_joint
- removed joint front_right_laser_joint
- removed joint front_right_middle_sonar_joint
- joint front_left_laser_joint: origin xyz=1 -2.3 0.5 rpy=0 0.05 0 -> xyz=0 -2.5 0.5 rpy=0 0 0

Commit message: Removing unused cameras

File: prius_description/urdf/prius.urdf (robot description, URDF)
Before this commit: robot prius, 14 links, 13 joints
Links:
- removed link back_camera_link
- removed link left_camera_link
- removed link right_camera_link
Joints:
- removed joint back_camera_joint
- removed joint left_camera_joint
- removed joint right_camera_joint

Commit message: Renaming left lidar -> central lidar

File: prius_description/urdf/prius.urdf (robot description, URDF)
Before this commit: robot prius, 11 links, 10 joints
Links:
- removed link front_left_laser_link
- added link front_central_laser_link, mass 1
Joints:
- removed joint front_left_laser_joint
- added joint front_central_laser_joint: type fixed, parent chassis, child front_central_laser_link, origin xyz=0 -2.4 0.4 rpy=0 0 -0.6707

Commit message: Prius.urdf updated for rviz/camera
Modifications made so that image can be visualized as Camera and laser can be overlayed.

File: prius_description/urdf/prius.urdf (robot description, URDF)
Before this commit: robot prius, 24 links, 23 joints
Links:
- added link back_camera_link_optical, mass 1
- added link front_camera_link_optical, mass 1
- added link left_camera_link_optical, mass 1
- added link right_camera_link_optical, mass 1
Joints:
- added joint back_camera_optical_joint: type fixed, parent back_camera_link, child back_camera_link_optical, origin xyz=0 0 0 rpy=-1.5707 0 -1.5707
- added joint front_camera_optical_joint: type fixed, parent front_camera_link, child front_camera_link_optical, origin xyz=0 0 0 rpy=-1.5707 0 -1.5707
- added joint left_camera_optical_joint: type fixed, parent left_camera_link, child left_camera_link_optical, origin xyz=0 0 0 rpy=-1.5707 0 -1.5707
- added joint right_camera_optical_joint: type fixed, parent right_camera_link, child right_camera_link_optical, origin xyz=0 0 0 rpy=-1.5707 0 -1.5707
